File: kicad/8x8_display.sch (KiCad schematic (older format))
At the start: 51 parts

Commit message: Finished schematic.
Parts:
- removed U?: 74HC238, symbol 74xx_IEEE:74HC238
- added C30: 20pF, symbol Device:C
- added R50: 100K, symbol Device:R
- added U1: 74HC08, symbol Local:74HC08
- added U26: 74HC238, symbol Local:74HC238
- gave numbers to parts that had none: 41
Connections:
- net DISP_ADDR_0: now also U26.1 (A0)
- net DISP_ADDR_1: now also U26.2 (A1)
- net DISP_ADDR_2: now also U26.3 (A2)
- net DRAW_PLAYER: now also U1.4
- net GND: now also C30.2, U26.4 (~G2A), U26.5 (~G2B), U26.8 (GND); no longer C17.1, C18.1, C19.1, C21.1, C22.1, C24.1, C25.2, C26.2, C27.1, C28.1, C29.2, C31.2, C32.2, R39.2, U15.16 (VCC), U16.16 (VCC), U17.16 (VCC), U18.16 (VCC), U19.4 (R), U19.8 (VCC), U20.16 (VCC), U21.14 (VCC), U22.16 (VCC), U23.16 (VCC), U24.16 (VCC), U25.16 (VCC), U28.14 (VCC), U29.14 (VCC)
- net RESET_5: now also U26.6 (G1)
- net at U10.1, U15.7 (QH), U16.7 (QH)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: now also U1.5
- net at U28.1: now also U26.7 (Y7)
- net at U28.3: now also U26.9 (Y6)
- net at U28.5: now also U26.10 (Y5)
- net at U28.9: now also U26.11 (Y4)
- net at U28.11: now also U26.12 (Y3)
- net at U28.13: now also U26.13 (Y2)
- net at U29.1: now also U26.14 (Y1)
- net at U29.3: now also U26.15 (Y0)
- new net: R50.2, U1.6
- new net COLLISION: C30.1, R50.1
- new net VCC: C17.1, C18.1, C19.1, C21.1, C22.1, C24.1, C25.2, C26.2, C27.1, C28.1, C29.2, C31.2, C32.2, R39.2, U15.16 (VCC), U16.16 (VCC), U17.16 (VCC), U18.16 (VCC), U19.4 (R), U19.8 (VCC), U20.16 (VCC), U21.14 (VCC), U22.16 (VCC), U23.16 (VCC), U24.16 (VCC), U25.16 (VCC), U26.16 (VCC), U28.14 (VCC), U29.14 (VCC)
- no-connect marks 1 -> 9
Other:
- moved on the sheet: C29

Commit message: KiCad: Added missing inverter on comparator output.
Parts:
- renumbered R39 to R40, R40 to R41, R41 to R42, R42 to R43, R43 to R44, R44 to R45, R45 to R46, R46 to R47, R47 to R48, R48 to R49, R49 to R50, R50 to R51, U28 to U15, U15 to U16, U16 to U17, U17 to U18, U18 to U19, U19 to U20, U20 to U21, U21 to U22, U22 to U23, U23 to U24, U24 to U25, U25 to U26, U26 to U27, U27 to U28, U28 to U29

Commit message: KiCad: Added opcode to enable/disable input and 64 respawn checkpoints.
Parts:
- added C20: 100nF, symbol Device:C
- added R31, R32, R33, R34, R35, R36, R37, R38: 100K, symbol Device:R
- added U20: 74HC244, symbol Local:74HC244
- C33: renamed from C30; value 20pF -> 47nF
- R50: renamed from R51; value 100K -> 10K
- renumbered C17 to C19, C18 to C21, C19 to C22, C20 to C23, C21 to C24, C22 to C25, C23 to C26, C24 to C27, C25 to C28, C26 to C29, C27 to C30, C28 to C31, C29 to C32, C31 to C34, C32 to C35, R40 to R39, R41 to R40, R42 to R41, R43 to R42, R44 to R43, R45 to R44, R46 to R45, R47 to R46, R48 to R47, R49 to R48, R50 to R49, U10 to U11, U15 to U16, U29 to U16, U16 to U18, U17 to U19, U1 to U2, U18 to U21, U19 to U22, U20 to U23, U21 to U24, U22 to U25, U23 to U26, U24 to U27, U25 to U28, U26 to U29, U27 to U30, U28 to U31, U29 to U32, U15 to U5
Connections:
- net COL_1: now also U20.2 (1A0); no longer U18.14 (SER)
- net COL_2: now also U20.4 (1A1); no longer U19.14 (SER)
- net COL_3: now also U20.6 (1A2); no longer U21.14 (SER)
- net COL_4: now also U20.8 (1A3); no longer U22.14 (SER)
- net COL_5: now also U20.17 (2A0); no longer U24.14 (SER)
- net COL_6: now also U20.15 (2A1); no longer U26.14 (SER)
- net COL_7: now also U20.13 (2A2); no longer U28.14 (SER)
- net COL_8: now also U20.11 (2A3); no longer U29.14 (SER)
- net GND: now also C20.1, R31.2, R32.2, R33.2, R34.2, R35.2, R36.2, R37.2, R38.2, U20.10 (GND)
- net VCC: now also C20.2, U20.20 (VCC)
- net Q7: now reaches U11.1, U18.7 (QH), U19.7 (QH), U2.5, U21.7 (QH), U22.7 (QH), U24.7 (QH), U26.7 (QH), U28.7 (QH), U29.7 (QH)
- net Q1: now reaches R43.2, U18.1 (QB), U19.1 (QB), U21.1 (QB), U22.1 (QB), U24.1 (QB), U26.1 (QB), U28.1 (QB), U29.1 (QB)
- net Q0: now reaches R42.2, U18.15 (QA), U19.15 (QA), U21.15 (QA), U22.15 (QA), U24.15 (QA), U26.15 (QA), U28.15 (QA), U29.15 (QA)
- net Q2: now reaches R44.2, U18.2 (QC), U19.2 (QC), U21.2 (QC), U22.2 (QC), U24.2 (QC), U26.2 (QC), U28.2 (QC), U29.2 (QC)
- net Q3: now reaches R45.2, U18.3 (QD), U19.3 (QD), U21.3 (QD), U22.3 (QD), U24.3 (QD), U26.3 (QD), U28.3 (QD), U29.3 (QD)
- net Q4: now reaches R46.2, U18.4 (QE), U19.4 (QE), U21.4 (QE), U22.4 (QE), U24.4 (QE), U26.4 (QE), U28.4 (QE), U29.4 (QE)
- net Q5: now reaches R47.2, U18.5 (QF), U19.5 (QF), U21.5 (QF), U22.5 (QF), U24.5 (QF), U26.5 (QF), U28.5 (QF), U29.5 (QF)
- net Q6: now reaches R48.2, U18.6 (QG), U19.6 (QG), U21.6 (QG), U22.6 (QG), U24.6 (QG), U26.6 (QG), U28.6 (QG), U29.6 (QG)
- new net: R34.1, U20.12 (1Y3), U22.14 (SER)
- new net: R35.1, U20.3 (2Y0), U24.14 (SER)
- new net: R36.1, U20.5 (2Y1), U26.14 (SER)
- new net: R31.1, U18.14 (SER), U20.18 (1Y0)
- new net: R32.1, U19.14 (SER), U20.16 (1Y1)
- new net: R33.1, U20.14 (1Y2), U21.14 (SER)
- new net: R37.1, U20.7 (2Y2), U28.14 (SER)
- new net: R38.1, U20.9 (2Y3), U29.14 (SER)
- new net ~INPUT_ENABLE: U20.1 (1OE), U20.19 (2OE)
Other:
- moved on the sheet: R49, U11A
