File: kicad/input.sch (KiCad schematic (older format))
At the start: 30 parts

Commit message: Finished schematic.
Parts:
- gave numbers to parts that had none: 6
- renumbered R1 to R19, R2 to R20, R3 to R21, R4 to R22, R5 to R23, R6 to R24, R7 to R25, R8 to R26, R9 to R27, R10 to R28, R11 to R29, R12 to R30, R13 to R31, R14 to R32, R15 to R33, R16 to R34
Connections:
- net GND: no longer U13.14 (GS)
- net VCC: no longer U13.15 (EO)
- no-connect marks 0 -> 2

Commit message: KiCad: Added missing inverter on comparator output.
Parts:
- added R35: 100K, symbol Device:R
- added U15: 74HC05, symbol Local:74HC05
Connections:
- net DRAW_PLAYER: now also R35.1, U15.6; no longer U14.19 (P=R)
- net VCC: now also R35.2
- new net: U14.19 (P=R), U15.5
Changed lines of the file:
@@
 Wire Wire Line
 	8400 2350 8775 2350
-Text HLabel 10200 2150 2    50   Output ~ 0
+Text HLabel 10450 2950 2    50   Output ~ 0
 DRAW_PLAYER
-Wire Wire Line
-	9775 2150 10200 2150
 Wire Wire Line
 	9275 4275 9275 4250
@@
 	1    0    0    -1
 $EndComp
+$Comp
+L Local:74HC05 U15
+U 3 1 5F3D2CBC
+P 10000 2550
+F 0 "U15" V 9954 2730 50  0000 L CNN
+F 1 "74HC05" V 10045 2730 50  0000 L CNN
+F 2 "" H 10000 2550 50  0001 C CNN
+F 3 "http://www.ti.com/lit/gpn/sn74HC05" H 10000 2550 50  0001 C CNN
+	3    10000 2550
+	0    1    1    0
+$EndComp
+$Comp
+L Device:R R35
+U 1 1 5F3EA3B4
+P 10000 3200
+F 0 "R35" H 10070 3246 50  0000 L CNN
+F 1 "100K" H 10070 3155 50  0000 L CNN
+F 2 "" V 9930 3200 50  0001 C CNN
+F 3 "~" H 10000 3200 50  0001 C CNN
+	1    10000 3200
+	1    0    0    -1
+$EndComp
+$Comp
+L power:VCC #PWR?
+U 1 1 5F3EA8F6
+P 10000 3575
+AR Path="/5F3EA8F6" Ref="#PWR?"  Part="1"
+AR Path="/5F587298/5F3EA8F6" Ref="#PWR036"  Part="1"
+F 0 "#PWR036" H 10000 3425 50  0001 C CNN
+F 1 "VCC" H 10017 3748 50  0000 C CNN
+F 2 "" H 10000 3575 50  0001 C CNN
+F 3 "" H 10000 3575 50  0001 C CNN
+	1    10000 3575
+	-1   0    0    1
+$EndComp
+Wire Wire Line
+	10000 3350 10000 3575
+Wire Wire Line
+	10000 2150 10000 2250
+Wire Wire Line
+	9775 2150 10000 2150
+Wire Wire Line
+	10450 2950 10000 2950
+Wire Wire Line
+	10000 2850 10000 2950
+Connection ~ 10000 2950
+Wire Wire Line
+	10000 2950 10000 3050
 $EndSCHEMATC

Commit message: KiCad: Added opcode to enable/disable input and 64 respawn checkpoints.
Parts:
- renumbered C12 to C14, C13 to C15, R19 to R10, R20 to R11, R21 to R12, R22 to R13, R23 to R14, R24 to R15, R25 to R16, R26 to R17, R27 to R18, R28 to R19, R29 to R20, R30 to R21, R31 to R22, R32 to R23, R33 to R24, R34 to R25, R35 to R26, U11 to U12, U12 to U13, U13 to U14, U14 to U15, U15 to U16
Connections:
- net GND: no longer U15.1 (G)
- new net ~ENABLE_OUTPUT: U15.1 (G)
