File: kicad/riverraid.sch (KiCad schematic (older format))
At the start: 42 parts

Commit message: Finished schematic.
Parts:
- added unit 5 of U4
- gave numbers to parts that had none: 40
Connections:
- net GND: now also C11.2, U9.32 (~CE), U9.34 (~OE); no longer C11.1
- net VCC: now also C11.1, U9.39 (~WE); no longer C11.2
- net at U2.13 (~R): now also U4.10
- new net 8x8 Matrix Display/COLLISION: U4.11
Other:
- moved on the sheet: C11

Commit message: KiCad: Added opcode to enable/disable input and 64 respawn checkpoints.
Parts:
- removed R10, R11, R12, R4, R5, R6, R7, R8, R9: 100K, symbol Device:R
- added C1, C8: 100nF, symbol Device:C
- added unit 1 of U1
- added unit 7 of U1
- added U5: 74HC05, symbol Local:74HC05
- renumbered C8 to C10, C9 to C11, C10 to C12, C11 to C13, C1 to C2, C2 to C3, C3 to C4, C4 to C5, C5 to C6, C6 to C7, C7 to C9, R13 to R4, R14 to R5, R15 to R6, R16 to R7, R17 to R8, R18 to R9, U4 to U1, U9 to U10, U10 to U11, U1 to U2, U2 to U3, U3 to U4, U5 to U6, U6 to U7, U7 to U8, U8 to U9
Connections:
- net GND: now also U6.1 (P1), U6.10 (P2), U6.15 (P0), U6.9 (P3), U7.1 (P1), U7.10 (P2), U7.15 (P0), U7.9 (P3), U8.1 (P1), U8.15 (P0), C1.1, C8.2, U1.7 (GND); no longer R3.2, R4.2, R5.2, R6.2, R7.2, R8.2, R9.2
- net VCC: now also R3.1, C1.2, U1.14 (VCC)
- net at U10.1 (A14), U9.7 (Q3): now also R6.1
- net at U10.2 (A12), U9.2 (Q1): now also R8.1
- net at U10.33 (A10), U8.7 (Q3): now also R4.1
- net at U10.35 (A11), U9.3 (Q0): now also R9.1
- net at U10.36 (A9), U8.6 (Q2): now also R5.1
- net at U10.38 (A13), U9.6 (Q2): now also R7.1
- net at U8.10 (P2): now also R5.2, U5.4; no longer R4.1
- net at U8.9 (P3): now also R4.2, U5.2; no longer R5.1
- net at U9.1 (P1): now also R8.2, U5.8; no longer R7.1
- net at U9.10 (P2): now also R7.2, U5.10; no longer R8.1
- net at U9.15 (P0): now also R9.2, U5.6; no longer R6.1
- net at U9.9 (P3): now also R6.2, U5.12; no longer R9.1
- net 8x8 Matrix Display/COL_1 renamed D0
- net 8x8 Matrix Display/COL_2 renamed D1
- net 8x8 Matrix Display/COL_3 renamed D2
- net 8x8 Matrix Display/COL_4 renamed D3
- net 8x8 Matrix Display/COL_5 renamed D4
- net 8x8 Matrix Display/COL_6 renamed D5
- net 8x8 Matrix Display/COL_7 renamed D6
- net 8x8 Matrix Display/COL_8 renamed D7
- new net: U1.2, U5.1, U5.11, U5.13, U5.3, U5.5, U5.9
- new net: C8.1, R3.2, U1.1
Other:
- moved on the sheet: C12, C2, C5, R4, R5, R6, R7, R8, R9, U1E, U1F, U2E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
